File: pcb/Buttons.kicad_sch (KiCad schematic)
At the start: 24 parts, among them SW1 SW_Push

Commit message: Updated footprints
Parts:
- removed C4 (x3): 220n, Capacitor_SMD:C_0603_1608Metric, symbol Device:C_Small
- removed R10 (x3): 10k, Resistor_SMD:R_0603_1608Metric, symbol Device:R
- removed R10: 110, Resistor_SMD:R_0603_1608Metric, symbol Device:R
- removed R10: 150, Resistor_SMD:R_0603_1608Metric, symbol Device:R
- removed R10 (x3): 36k, Resistor_SMD:R_0603_1608Metric, symbol Device:R
- removed R10: 120, Resistor_SMD:R_0603_1608Metric, symbol Device:R
- added C4 (x3): 220n, Capacitor_SMD:C_1206_3216Metric, symbol Device:C_Small
- added R10 (x3): 36k, Resistor_SMD:R_1206_3216Metric, symbol Device:R
- added R10 (x3): 10k, Resistor_SMD:R_1206_3216Metric, symbol Device:R
- added R10: 150, Resistor_SMD:R_1206_3216Metric, symbol Device:R
- added R10: 110, Resistor_SMD:R_1206_3216Metric, symbol Device:R
- added R10: 120, Resistor_SMD:R_1206_3216Metric, symbol Device:R
- C4: footprint Capacitor_SMD:C_0603_1608Metric -> Capacitor_SMD:C_1206_3216Metric
- D10, D11, D12, D13: footprint (none) -> LED_SMD:LED_1206_3216Metric
- R10: footprint Resistor_SMD:R_0603_1608Metric -> Resistor_SMD:R_1206_3216Metric
- SW1: footprint (none) -> Button_Switch_THT:SW_PUSH_6mm_H4.3mm
Connections:
- net +3.3V: now also R10.1, R10.1, R10.1
- net GND: now also C4.2, C4.2, C4.2
- net MCU_Button2: now also C4.1, R10.2
- net MCU_Button3: now also C4.1, R10.2
- net MCU_Button4: now also C4.1, R10.2
- net MCU_LED_Gelb: now also R10.1
- net MCU_LED_Green1: now also R10.1
- net MCU_LED_Red: now also R10.1
- net at SW1.1: now also R10.1, R10.2 (x3)
- net at D13.2 (A): now also R10.2
- net at D10.2 (A): now also R10.2
- net at D12.2 (A): now also R10.2

Commit message: updated pcb
Parts:
- removed C4 (x2): 220n, Capacitor_SMD:C_1206_3216Metric, symbol Device:C_Small
- removed R10 (x2): 36k, Resistor_SMD:R_1206_3216Metric, symbol Device:R
- removed R10 (x2): 10k, Resistor_SMD:R_1206_3216Metric, symbol Device:R
- removed SW1 (x4): SW_Push, Button_Switch_THT:SW_PUSH_6mm_H4.3mm, symbol Switch:SW_Push
- added C4: 220n, Capacitor_SMD:C_1206_3216Metric, symbol Device:C_Small
- added D14, D15: LED_Gelb, LED_SMD:LED_1206_3216Metric, symbol Device:LED
- added D16: LED_Green, LED_SMD:LED_1206_3216Metric, symbol Device:LED
- added J1, J6, J7, J8: Conn_01x02_Pin, Connector_PinHeader_2.54mm:PinHeader_2x01_P2.54mm_Vertical_SMD, symbol Connector:Conn_01x02_Pin
- added R10 (x2): 120, Resistor_SMD:R_1206_3216Metric, symbol Device:R
- added R10 (x2): 10k, Resistor_SMD:R_1206_3216Metric, symbol Device:R
- added R10: 150, Resistor_SMD:R_1206_3216Metric, symbol Device:R
- added R10: 36k, Resistor_SMD:R_1206_3216Metric, symbol Device:R
Connections:
- net +3.3V: now also J1.1 (Pin_1), R10.1
- net GND: now also C4.2, D14.1 (K), D15.1 (K), D16.1 (K), J6.2 (Pin_2), J7.2 (Pin_2), J8.2 (Pin_2), R10.1
- net at R10.1, R10.2: now also J8.1 (Pin_1)
- net at R10.1, R10.2: now also J7.1 (Pin_1)
- net MCU_Button1 renamed MCU_Vorfahren
- net MCU_Button2 renamed MCU_Zurueckfahren
- net MCU_LED_Gelb renamed MCU_LED_Manuell
- net MCU_LED_Green1 renamed MCU_LED_PWR
- net MCU_LED_Green2 renamed MCU_LED_Betrieb
- net MCU_LED_Red renamed MCU_LED_Stoerung
- new net: J6.1 (Pin_1), R10.1, R10.2
- new net: D14.2 (A), R10.2
- new net: D16.2 (A), R10.2
- new net: D15.2 (A), R10.2
- new net MCU_Kalibrierung: C4.1, R10.2
- new net MCU_LED_Kalibrierung: R10.1
- new net MCU_LED_Rollen: R10.1
- new net MCU_LED_Trimmen: R10.1
- new net MCU_Switch: J1.2 (Pin_2), R10.2
