File: pcb/Endschalter.kicad_sch (KiCad schematic)
At the start: 4 parts

Commit message: Updated footprints
Parts:
- Enschalter_Hinten_1, Enschalter_Vorne_1: footprint (none) -> Connector_Phoenix_MSTB:PhoenixContact_MSTBA_2,5_4-G-5,08_1x04_P5.08mm_Horizontal
Changed lines of the file:
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@@
       (effects (font (size 1.27 1.27)))
     )
-    (property "Footprint" "" (at 31.75 46.99 0)
+    (property "Footprint" "Connector_Phoenix_MSTB:PhoenixContact_MSTBA_2,5_4-G-5,08_1x04_P5.08mm_Horizontal" (at 31.75 46.99 0)
       (effects (font (size 1.27 1.27)) hide)
     )
@@
       (effects (font (size 1.27 1.27)))
     )
-    (property "Footprint" "" (at 31.75 31.75 0)
+    (property "Footprint" "Connector_Phoenix_MSTB:PhoenixContact_MSTBA_2,5_4-G-5,08_1x04_P5.08mm_Horizontal" (at 31.75 31.75 0)
       (effects (font (size 1.27 1.27)) hide)
     )

Commit message: updated pcb
Parts:
- removed Enschalter_Hinten_1, Enschalter_Vorne_1: Conn_01x04_Pin, Connector_Phoenix_MSTB:PhoenixContact_MSTBA_2,5_4-G-5,08_1x04_P5.08mm_Horizontal, symbol Connector:Conn_01x04_Pin
- added Endschalter_Hinten1, Endschalter_Vorne1: Conn_01x03_Pin, TerminalBlock_TE-Connectivity:TerminalBlock_TE_282834-3_1x03_P2.54mm_Horizontal, symbol Connector:Conn_01x03_Pin
- D1, D2: footprint Diode_SMD:D_SMB -> Diode_SMD:D_SOD-123
Connections:
- net +24V: now also Endschalter_Hinten1.1 (Pin_1), Endschalter_Vorne1.1 (Pin_1)
- net GND: now also Endschalter_Hinten1.2 (Pin_2), Endschalter_Vorne1.2 (Pin_2)
- net Endschalter_Hinten_IN_1 renamed Endschalter_Hinten
- net Endschalter_Hinten: now also Endschalter_Hinten1.3 (Pin_3)
- net Endschalter_Vorne_IN_1 renamed Endschalter_Vorne
- net Endschalter_Vorne: now also Endschalter_Vorne1.3 (Pin_3)
- no-connect marks 2 -> 0
Changed lines of the file:
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@@
 (kicad_sch (version 20230121) (generator eeschema)
   (paper "A4")
-  (junction (at 53.34 49.53) (diameter 0) (color 0 0 0 0)
+  (junction (at 46.99 31.75) (diameter 0) (color 0 0 0 0)
   )
   (junction (at 63.5 36.83) (diameter 0) (color 0 0 0 0)
@@
   (junction (at 63.5 52.07) (diameter 0) (color 0 0 0 0)
   )
-  (junction (at 46.99 29.21) (diameter 0) (color 0 0 0 0)
-  )
-  (no_connect (at 36.83 31.75))
-  (no_connect (at 36.83 46.99))
-  (wire (pts (xy 36.83 29.21) (xy 46.99 29.21))
-    (stroke (width 0) (type default))
-  )
-  (wire (pts (xy 53.34 34.29) (xy 53.34 49.53))
+  (junction (at 50.8 49.53) (diameter 0) (color 0 0 0 0)
+  )
+  (wire (pts (xy 50.8 34.29) (xy 50.8 49.53))
     (stroke (width 0) (type default))
   )
@@
     (stroke (width 0) (type default))
   )
-  (wire (pts (xy 53.34 49.53) (xy 53.34 58.42))
-    (stroke (width 0) (type default))
-  )
-  (wire (pts (xy 36.83 52.07) (xy 63.5 52.07))
-    (stroke (width 0) (type default))
-  )
-  (wire (pts (xy 36.83 36.83) (xy 63.5 36.83))
-    (stroke (width 0) (type default))
-  )
-  (wire (pts (xy 46.99 44.45) (xy 46.99 29.21))
-    (stroke (width 0) (type default))
-  )
-  (wire (pts (xy 36.83 44.45) (xy 46.99 44.45))
-    (stroke (width 0) (type default))
-  )
-  (wire (pts (xy 36.83 34.29) (xy 53.34 34.29))
+  (wire (pts (xy 34.29 34.29) (xy 50.8 34.29))
+    (stroke (width 0) (type default))
+  )
+  (wire (pts (xy 50.8 49.53) (xy 50.8 58.42))
+    (stroke (width 0) (type default))
+  )
+  (wire (pts (xy 34.29 52.07) (xy 63.5 52.07))
+    (stroke (width 0) (type default))
+  )
+  (wire (pts (xy 34.29 36.83) (xy 63.5 36.83))
+    (stroke (width 0) (type default))
+  )
+  (wire (pts (xy 46.99 46.99) (xy 46.99 31.75))
     (stroke (width 0) (type default))
   )
@@
     (stroke (width 0) (type default))
   )
-  (wire (pts (xy 36.83 49.53) (xy 53.34 49.53))
-    (stroke (width 0) (type default))
-  )
-  (wire (pts (xy 46.99 27.94) (xy 46.99 29.21))
+  (wire (pts (xy 34.29 49.53) (xy 50.8 49.53))
+    (stroke (width 0) (type default))
+  )
+  (wire (pts (xy 34.29 31.75) (xy 46.99 31.75))
+    (stroke (width 0) (type default))
+  )
+  (wire (pts (xy 46.99 27.94) (xy 46.99 31.75))
     (stroke (width 0) (type default))
   )
@@
     (stroke (width 0) (type default))
   )
+  (wire (pts (xy 46.99 46.99) (xy 34.29 46.99))
+    (stroke (width 0) (type default))
+  )
   (wire (pts (xy 63.5 44.45) (xy 63.5 43.18))
     (stroke (width 0) (type default))
   )
-  (hierarchical_label "Endschalter_Hinten_IN_1" (shape output) (at 83.82 52.07 0) (fields_autoplaced)
+  (hierarchical_label "Endschalter_Hinten" (shape output) (at 83.82 52.07 0) (fields_autoplaced)
     (effects (font (size 1.27 1.27)) (justify left))
   )
-  (hierarchical_label "Endschalter_Vorne_IN_1" (shape output) (at 83.82 36.83 0) (fields_autoplaced)
+  (hierarchical_label "Endschalter_Vorne" (shape output) (at 83.82 36.83 0) (fields_autoplaced)
     (effects (font (size 1.27 1.27)) (justify left))
+  )
+  (symbol (lib_id "Connector:Conn_01x03_Pin") (at 29.21 34.29 0) (unit 1)
+    (in_bom yes) (on_board yes) (dnp no)
+    (property "Reference" "Endschalter_Vorne1" (at 30.48 26.67 0)
+      (effects (font (size 1.27 1.27)))
+    )
+    (property "Value" "Conn_01x03_Pin" (at 30.48 29.21 0)
+      (effects (font (size 1.27 1.27)))
+    )
+    (property "Footprint" "TerminalBlock_TE-Connectivity:TerminalBlock_TE_282834-3_1x03_P2.54mm_Horizontal" (at 29.21 34.29 0)
+      (effects (font (size 1.27 1.27)) hide)
+    )
+    (property "Datasheet" "~" (at 29.21 34.29 0)
+      (effects (font (size 1.27 1.27)) hide)
+    )
+    (pin "1")
+    (pin "2")
+    (pin "3")
+    (instances
+      (project "STM32_F439ZI_Shield"
+        (path "/19bff231-ff37-4a40-bd06-2039e9f55c77/d69a8748-4c21-4b63-b4ce-9072d526117b"
+          (reference "Endschalter_Vorne1") (unit 1)
+        )
+      )
+    )
   )
   (symbol (lib_id "power:+24V") (at 46.99 27.94 0) (unit 1)
@@
       (effects (font (size 1.27 1.27)) (justify left))
     )
-    (property "Footprint" "Diode_SMD:D_SMB" (at 59.055 40.64 0)
+    (property "Footprint" "Diode_SMD:D_SOD-123" (at 59.055 40.64 0)
       (effects (font (size 1.27 1.27)) hide)
     )
@@
     )
   )
-  (symbol (lib_id "power:GND") (at 53.34 58.42 0) (unit 1)
-    (in_bom yes) (on_board yes) (dnp no)
-    (property "Reference" "#PWR03" (at 53.34 64.77 0)
-      (effects (font (size 1.27 1.27)) hide)
-    )
-    (property "Value" "GND" (at 53.34 62.23 0)
-      (effects (font (size 1.27 1.27)))
-    )
-    (property "Footprint" "" (at 53.34 58.42 0)
-      (effects (font (size 1.27 1.27)) hide)
-    )
-    (property "Datasheet" "" (at 53.34 58.42 0)
+  (symbol (lib_id "power:GND") (at 50.8 58.42 0) (unit 1)
+    (in_bom yes) (on_board yes) (dnp no)
+    (property "Reference" "#PWR03" (at 50.8 64.77 0)
+      (effects (font (size 1.27 1.27)) hide)
+    )
+    (property "Value" "GND" (at 50.8 62.23 0)
+      (effects (font (size 1.27 1.27)))
+    )
+    (property "Footprint" "" (at 50.8 58.42 0)
+      (effects (font (size 1.27 1.27)) hide)
+    )
+    (property "Datasheet" "" (at 50.8 58.42 0)
       (effects (font (size 1.27 1.27)) hide)
     )
@@
         (path "/19bff231-ff37-4a40-bd06-2039e9f55c77/d69a8748-4c21-4b63-b4ce-9072d526117b"
           (reference "#PWR05") (unit 1)
-        )
-      )
-    )
-  )
-  (symbol (lib_id "Connector:Conn_01x04_Pin") (at 31.75 46.99 0) (unit 1)
-    (in_bom yes) (on_board yes) (dnp no)
-    (property "Reference" "Enschalter_Hinten_1" (at 34.29 55.88 0)
-      (effects (font (size 1.27 1.27)))
-    )
-    (property "Value" "Conn_01x04_Pin" (at 34.29 53.34 0)
-      (effects (font (size 1.27 1.27)))
-    )
-    (property "Footprint" "Connector_Phoenix_MSTB:PhoenixContact_MSTBA_2,5_4-G-5,08_1x04_P5.08mm_Horizontal" (at 31.75 46.99 0)
-      (effects (font (size 1.27 1.27)) hide)
-    )
-    (property "Datasheet" "~" (at 31.75 46.99 0)
-      (effects (font (size 1.27 1.27)) hide)
-    )
-    (pin "1")
-    (pin "2")
-    (pin "3")
-    (pin "4")
-    (instances
-      (project "STM32_F439ZI_Shield"
-        (path "/19bff231-ff37-4a40-bd06-2039e9f55c77"
-          (reference "Enschalter_Hinten_1") (unit 1)
-        )
-        (path "/19bff231-ff37-4a40-bd06-2039e9f55c77/d69a8748-4c21-4b63-b4ce-9072d526117b"
-          (reference "Enschalter_Hinten_1") (unit 1)
         )
       )
@@
       (effects (font (size 1.27 1.27)) (justify left))
     )
-    (property "Footprint" "Diode_SMD:D_SMB" (at 59.055 55.88 0)
+    (property "Footprint" "Diode_SMD:D_SOD-123" (at 59.055 55.88 0)
       (effects (font (size 1.27 1.27)) hide)
     )
@@
     )
   )
-  (symbol (lib_id "Connector:Conn_01x04_Pin") (at 31.75 31.75 0) (unit 1)
-    (in_bom yes) (on_board yes) (dnp no)
-    (property "Reference" "Enschalter_Vorne_1" (at 34.29 40.64 0)
-      (effects (font (size 1.27 1.27)))
-    )
-    (property "Value" "Conn_01x04_Pin" (at 34.29 38.1 0)
-      (effects (font (size 1.27 1.27)))
-    )
-    (property "Footprint" "Connector_Phoenix_MSTB:PhoenixContact_MSTBA_2,5_4-G-5,08_1x04_P5.08mm_Horizontal" (at 31.75 31.75 0)
-      (effects (font (size 1.27 1.27)) hide)
-    )
-    (property "Datasheet" "~" (at 31.75 31.75 0)
+  (symbol (lib_id "Connector:Conn_01x03_Pin") (at 29.21 49.53 0) (unit 1)
+    (in_bom yes) (on_board yes) (dnp no)
+    (property "Reference" "Endschalter_Hinten1" (at 33.02 41.91 0)
+      (effects (font (size 1.27 1.27)))
+    )
+    (property "Value" "Conn_01x03_Pin" (at 33.02 44.45 0)
+      (effects (font (size 1.27 1.27)))
+    )
+    (property "Footprint" "TerminalBlock_TE-Connectivity:TerminalBlock_TE_282834-3_1x03_P2.54mm_Horizontal" (at 29.21 49.53 0)
+      (effects (font (size 1.27 1.27)) hide)
+    )
+    (property "Datasheet" "~" (at 29.21 49.53 0)
       (effects (font (size 1.27 1.27)) hide)
     )
@@
     (pin "2")
     (pin "3")
-    (pin "4")
-    (instances
-      (project "STM32_F439ZI_Shield"
-        (path "/19bff231-ff37-4a40-bd06-2039e9f55c77"
-          (reference "Enschalter_Vorne_1") (unit 1)
-        )
-        (path "/19bff231-ff37-4a40-bd06-2039e9f55c77/d69a8748-4c21-4b63-b4ce-9072d526117b"
-          (reference "Enschalter_Vorne_1") (unit 1)
-        )
-      )
+    (instances
+      (project "STM32_F439ZI_Shield"
+        (path "/19bff231-ff37-4a40-bd06-2039e9f55c77/d69a8748-4c21-4b63-b4ce-9072d526117b"
+          (reference "Endschalter_Hinten1") (unit 1)
+        )
+      )
