File: pcb/untitled.kicad_sch (KiCad schematic)
At the start: 27 parts, among them U3 VO618A

Commit message: Updated footprints
Parts:
- removed R10 (x4): 2,2k, Resistor_SMD:R_0603_1608Metric, symbol Device:R
- removed R10 (x3): 700, Resistor_SMD:R_0603_1608Metric, symbol Device:R
- removed R8 (x4): 6,6k, Resistor_SMD:R_0201_0603Metric, symbol Device:R
- removed R8 (x3): 11k, Resistor_SMD:R_0201_0603Metric, symbol Device:R
- removed U3 (x9): VO618A, Package_DIP:DIP-4_W7.62mm, symbol Isolator:VO615A
- added R10 (x3): 700, Resistor_SMD:R_1206_3216Metric, symbol Device:R
- added R10 (x4): 2,2k, Resistor_SMD:R_1206_3216Metric, symbol Device:R
- added R8 (x3): 11k, Resistor_SMD:R_1206_3216Metric, symbol Device:R
- added R8 (x4): 6,8k, Resistor_SMD:R_1206_3216Metric, symbol Device:R
- added U10, U11, U3, U4, U5, U6, U7, U8, U9: LTV-817S, Package_DIP:SMDIP-4_W9.53mm, symbol Isolator:LTV-817S
- R10: footprint Resistor_SMD:R_0603_1608Metric -> Resistor_SMD:R_1206_3216Metric
- R8: value 6,6k -> 6,8k; footprint Resistor_SMD:R_0201_0603Metric -> Resistor_SMD:R_1206_3216Metric
- R8: footprint Resistor_SMD:R_0201_0603Metric -> Resistor_SMD:R_1206_3216Metric
Connections:
- net +24V: now also U3.4, U4.4, U5.4, U6.4
- net +3.3V: now also U10.4, U11.4, U7.4, U8.4, U9.4
- net Endschalter_Hinten_MCU: now also U11.3
- net Endschalter_Vorne_HV_IN: now also R10.1
- net Endschalter_Vorne_MCU: now also R8.1, U10.3
- net GND: now also R8.2, R8.2, R8.2, R8.2, R8.2, R8.2, R8.2, U10.2, U11.2, U3.2, U4.2, U5.2, U6.2, U7.2, U8.2, U9.2
- net IN0_HV: now also U3.3
- net IN1_MCU_IN: now also R10.1
- net IN2_HV: now also R8.1, U5.3
- net IN2_MCU_IN: now also R10.1
- net IN3_HV: now also R8.1, U6.3
- net IN3_MCU_IN: now also R10.1
- net OUT1_HV_IN: now also R10.1
- net OUT1_MCU: now also R8.1, U7.3
- net OUT2_HV_IN: now also R10.1
- net OUT2_MCU: now also R8.1, U8.3
- net OUT3_HV_IN: now also R10.1
- net OUT3_MCU: now also R8.1, U9.3
- net at R10.2: now also U11.1
- net at R10.2: now also U3.1
- new net: R10.2, U5.1
- new net: R10.2, U9.1
- new net: R10.2, U6.1
- new net: R10.2, U4.1
- new net: R8.1, U4.3
- new net: R10.2, U7.1
- new net: R10.2, U8.1
- new net: R10.2, U10.1

Commit message: updated pcb
Parts:
- removed R10 (x2): 2,2k, Resistor_SMD:R_1206_3216Metric, symbol Device:R
- removed R8 (x2): 6,8k, Resistor_SMD:R_1206_3216Metric, symbol Device:R
- added R10 (x2): 700, Resistor_SMD:R_1206_3216Metric, symbol Device:R
- added R8 (x2): 11k, Resistor_SMD:R_1206_3216Metric, symbol Device:R
Connections:
- net +24V: now also U10.4, U11.4
- net +3.3V: no longer U10.4, U11.4
- net GND: now also R8.2, R8.2
- net at U11.1: now also R10.2
- net IN1_HV: now reaches R8.1, U4.3
- net at U10.1: now also R10.2
- net Endschalter_Hinten_MCU renamed Ext_Relais2_OUT
- net Ext_Relais2_OUT: now also R8.1
- net Endschalter_Vorne_MCU renamed Ext_Relais1_OUT
- net Ext_Relais1_OUT: now also R8.1
- new net Ext_Relais1_MCU: R10.1
- new net Ext_Relais2_MCU: R10.1
