File: pcb/Motor.kicad_sch (KiCad schematic)
At the start: 7 parts

Commit message: Updated PCB
Parts:
- added D2 (x3): SMPJ5359B-TP, Diode_SMD:D_SMB, symbol Diode:Z2SMBxxx
Connections:
- net GND: now also Motor_Logik_1.8 (Pin_8), D2.2 (A), D2.2 (A), D2.2 (A)
- net OUT1_IN: now reaches Motor_Logik_1.10 (Pin_10)
- net OUT1_IN: now also D2.1 (K)
- net OUT2_IN: now reaches Motor_Logik_1.11 (Pin_11)
- net OUT2_IN: now also D2.1 (K)
- net OUT3_IN: now reaches Motor_Logik_1.12 (Pin_12)
- net OUT3_IN: now also D2.1 (K)
- net Drehzahl_Analog_OUT: now reaches Motor_Logik_1.7 (Pin_7)
- net +24V: now reaches Motor_Logik_1.9 (Pin_9)

Commit message: updated pcb
Parts:
- added U12: TMCS1101A2BQDR, SOIC_D_8_TEX, symbol TMCS:PMCS1101A1BQDR
Connections:
- net +24V: now also U12.1 (IN+), U12.2 (IN+)
- net GND: now also Motor_Leistungsversorgung_1.3 (Pin_3), U12.5 (GND)
- net at F2.2: now also U12.3 (IN-), U12.4 (IN-)
- new net +3.3V: U12.8 (VS)
- new net Stromsensor_MCU: U12.7 (VOUT)
- no-connect marks 3 -> 4
Changed lines of the file:
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@@
   (junction (at 107.95 55.88) (diameter 0) (color 0 0 0 0)
   )
+  (junction (at 50.8 30.48) (diameter 0) (color 0 0 0 0)
+  )
+  (junction (at 50.8 25.4) (diameter 0) (color 0 0 0 0)
+  )
   (junction (at 125.73 60.96) (diameter 0) (color 0 0 0 0)
   )
@@
   )
   (no_connect (at 83.82 66.04))
+  (no_connect (at 77.47 29.21))
   (no_connect (at 29.21 33.02))
   (no_connect (at 83.82 68.58))
@@
     (stroke (width 0) (type default))
   )
+  (wire (pts (xy 50.8 25.4) (xy 50.8 26.67))
+    (stroke (width 0) (type default))
+  )
   (wire (pts (xy 116.84 58.42) (xy 134.62 58.42))
     (stroke (width 0) (type default))
   )
-  (wire (pts (xy 44.45 30.48) (xy 45.72 30.48))
+  (wire (pts (xy 29.21 35.56) (xy 44.45 35.56))
     (stroke (width 0) (type default))
   )
@@
     (stroke (width 0) (type default))
   )
+  (wire (pts (xy 50.8 30.48) (xy 50.8 31.75))
+    (stroke (width 0) (type default))
+  )
+  (wire (pts (xy 50.8 24.13) (xy 50.8 25.4))
+    (stroke (width 0) (type default))
+  )
+  (wire (pts (xy 77.47 26.67) (xy 80.01 26.67))
+    (stroke (width 0) (type default))
+  )
   (wire (pts (xy 125.73 85.09) (xy 125.73 82.55))
     (stroke (width 0) (type default))
@@
     (stroke (width 0) (type default))
   )
+  (wire (pts (xy 44.45 35.56) (xy 44.45 36.83))
+    (stroke (width 0) (type default))
+  )
   (wire (pts (xy 33.02 58.42) (xy 48.26 58.42))
     (stroke (width 0) (type default))
   )
+  (wire (pts (xy 50.8 29.21) (xy 50.8 30.48))
+    (stroke (width 0) (type default))
+  )
   (wire (pts (xy 58.42 60.96) (xy 58.42 68.58))
     (stroke (width 0) (type default))
   )
-  (wire (pts (xy 29.21 35.56) (xy 45.72 35.56))
-    (stroke (width 0) (type default))
-  )
   (wire (pts (xy 107.95 55.88) (xy 107.95 74.93))
     (stroke (width 0) (type default))
@@
     (stroke (width 0) (type default))
   )
-  (wire (pts (xy 45.72 35.56) (xy 45.72 36.83))
-    (stroke (width 0) (type default))
-  )
   (wire (pts (xy 96.52 63.5) (xy 160.02 63.5))
     (stroke (width 0) (type default))
@@
     (stroke (width 0) (type default))
   )
+  (wire (pts (xy 77.47 24.13) (xy 80.01 24.13))
+    (stroke (width 0) (type default))
+  )
   (wire (pts (xy 107.95 55.88) (xy 134.62 55.88))
     (stroke (width 0) (type default))
   )
+  (wire (pts (xy 46.99 25.4) (xy 50.8 25.4))
+    (stroke (width 0) (type default))
+  )
   (wire (pts (xy 96.52 68.58) (xy 134.62 68.58))
+    (stroke (width 0) (type default))
+  )
+  (wire (pts (xy 44.45 30.48) (xy 50.8 30.48))
     (stroke (width 0) (type default))
   )
@@
     (effects (font (size 1.27 1.27)) (justify left))
   )
+  (hierarchical_label "Stromsensor_MCU" (shape output) (at 80.01 26.67 0) (fields_autoplaced)
+    (effects (font (size 1.27 1.27)) (justify left))
+  )
   (hierarchical_label "IN0_OUT" (shape input) (at 33.02 55.88 180) (fields_autoplaced)
     (effects (font (size 1.27 1.27)) (justify right))
@@
   (hierarchical_label "IN3_OUT" (shape input) (at 33.02 63.5 180) (fields_autoplaced)
     (effects (font (size 1.27 1.27)) (justify right))
+  )
+  (symbol (lib_id "TMCS:PMCS1101A1BQDR") (at 36.83 24.13 0) (unit 1)
+    (in_bom yes) (on_board yes) (dnp no)
+    (property "Reference" "U12" (at 64.77 17.78 0)
+      (effects (font (size 1.524 1.524)))
+    )
+    (property "Value" "TMCS1101A2BQDR" (at 64.77 20.32 0)
+      (effects (font (size 1.524 1.524)))
+    )
+    (property "Footprint" "SOIC_D_8_TEX" (at 63.5 20.32 0)
+      (effects (font (size 1.524 1.524)) hide)
+    )
+    (property "Datasheet" "" (at 50.8 24.13 0)
+      (effects (font (size 1.524 1.524)))
+    )
+    (pin "1")
+    (pin "2")
+    (pin "3")
+    (pin "4")
+    (pin "5")
+    (pin "6")
+    (pin "7")
+    (pin "8")
+    (instances
+      (project "STM32_F439ZI_Shield"
+        (path "/19bff231-ff37-4a40-bd06-2039e9f55c77"
+          (reference "U12") (unit 1)
+        )
+        (path "/19bff231-ff37-4a40-bd06-2039e9f55c77/3e3b4274-21ab-4d07-973d-ec15fa140762"
+          (reference "U12") (unit 1)
+        )
+      )
+    )
   )
   (symbol (lib_id "power:+24V") (at 160.02 63.5 0) (unit 1)
@@
         (path "/19bff231-ff37-4a40-bd06-2039e9f55c77/3e3b4274-21ab-4d07-973d-ec15fa140762"
           (reference "F2") (unit 1)
+        )
+      )
+    )
+  )
+  (symbol (lib_id "power:GND") (at 77.47 31.75 0) (unit 1)
+    (in_bom yes) (on_board yes) (dnp no)
+    (property "Reference" "#PWR062" (at 77.47 38.1 0)
+      (effects (font (size 1.27 1.27)) hide)
+    )
+    (property "Value" "GND" (at 77.47 35.56 0)
+      (effects (font (size 1.27 1.27)))
+    )
+    (property "Footprint" "" (at 77.47 31.75 0)
+      (effects (font (size 1.27 1.27)) hide)
+    )
+    (property "Datasheet" "" (at 77.47 31.75 0)
+      (effects (font (size 1.27 1.27)) hide)
+    )
+    (pin "1")
+    (instances
+      (project "STM32_F439ZI_Shield"
+        (path "/19bff231-ff37-4a40-bd06-2039e9f55c77/3e3b4274-21ab-4d07-973d-ec15fa140762"
+          (reference "#PWR062") (unit 1)
         )
       )
@@
     )
   )
+  (symbol (lib_id "power:GND") (at 44.45 36.83 0) (unit 1)
+    (in_bom yes) (on_board yes) (dnp no)
+    (property "Reference" "#PWR064" (at 44.45 43.18 0)
+      (effects (font (size 1.27 1.27)) hide)
+    )
+    (property "Value" "GND" (at 44.45 40.64 0)
+      (effects (font (size 1.27 1.27)))
+    )
+    (property "Footprint" "" (at 44.45 36.83 0)
+      (effects (font (size 1.27 1.27)) hide)
+    )
+    (property "Datasheet" "" (at 44.45 36.83 0)
+      (effects (font (size 1.27 1.27)) hide)
+    )
+    (pin "1")
+    (instances
+      (project "STM32_F439ZI_Shield"
+        (path "/19bff231-ff37-4a40-bd06-2039e9f55c77/3e3b4274-21ab-4d07-973d-ec15fa140762"
+          (reference "#PWR064") (unit 1)
+        )
+      )
+    )
+  )
   (symbol (lib_id "Connector:Conn_01x03_Pin") (at 24.13 33.02 0) (unit 1)
     (in_bom yes) (on_board yes) (dnp no)
@@
     )
   )
+  (symbol (lib_id "power:+3.3V") (at 80.01 24.13 0) (unit 1)
+    (in_bom yes) (on_board yes) (dnp no) (fields_autoplaced)
+    (property "Reference" "#PWR063" (at 80.01 27.94 0)
+      (effects (font (size 1.27 1.27)) hide)
+    )
+    (property "Value" "+3.3V" (at 80.01 20.32 0)
+      (effects (font (size 1.27 1.27)))
+    )
+    (property "Footprint" "" (at 80.01 24.13 0)
+      (effects (font (size 1.27 1.27)) hide)
+    )
+    (property "Datasheet" "" (at 80.01 24.13 0)
+      (effects (font (size 1.27 1.27)) hide)
+    )
+    (pin "1")
+    (instances
+      (project "STM32_F439ZI_Shield"
+        (path "/19bff231-ff37-4a40-bd06-2039e9f55c77/3e3b4274-21ab-4d07-973d-ec15fa140762"
+          (reference "#PWR063") (unit 1)
+        )
+      )
+    )
+  )
   (symbol (lib_id "power:GND") (at 39.37 78.74 0) (unit 1)
     (in_bom yes) (on_board yes) (dnp no)
@@
         )
       )
+    )
+  )
+  (symbol (lib_id "power:+24V") (at 46.99 25.4 0) (unit 1)
+    (in_bom yes) (on_board yes) (dnp no) (fields_autoplaced)
+    (property "Reference" "#PWR065" (at 46.99 29.21 0)
+      (effects (font (size 1.27 1.27)) hide)
+    )
+    (property "Value" "+24V" (at 46.99 21.59 0)
+      (effects (font (size 1.27 1.27)))
+    )
+    (property "Footprint" "" (at 46.99 25.4 0)
+      (effects (font (size 1.27 1.27)) hide)
+    )
+    (property "Datasheet" "" (at 46.99 25.4 0)
+      (effects (font (size 1.27 1.27)) hide)
+    )
+    (pin "1")
+    (instances
+      (project "STM32_F439ZI_Shield"
+        (path "/19bff231-ff37-4a40-bd06-2039e9f55c77/3e3b4274-21ab-4d07-973d-ec15fa140762"
+          (reference "#PWR065") (unit 1)
+        )
+      )

Commit message: Updated footprints
Parts:
- removed U12: TMCS1101A2BQDR, SOIC_D_8_TEX, symbol TMCS:PMCS1101A1BQDR
- added U15: ACS724xLCTR-05AB, Package_SO:SOIC-8_3.9x4.9mm_P1.27mm, symbol Sensor_Current:ACS724xLCTR-05AB
- F2: footprint (none) -> Fuse:Fuse_BelFuse_0ZRE0005FF_L8.3mm_W3.8mm
- Motor_Leistungsversorgung_1: footprint (none) -> Connector_Phoenix_MSTB:PhoenixContact_MSTBA_2,5_3-G_1x03_P5.00mm_Horizontal
- Motor_Logik_1: footprint (none) -> Connector_PinHeader_2.54mm:PinHeader_2x06_P2.54mm_Vertical_SMD
Connections:
- net +24V: now also U15.1 (IP+), U15.2 (IP+)
- net GND: now also U15.5 (GND)
- net Stromsensor_MCU: now also U15.7 (VIOUT)
- net at F2.2: now also U15.3 (IP-), U15.4 (IP-)
- new net +5V: U15.8 (VCC)

Commit message: updated pcb
Parts:
- removed Motor_Leistungsversorgung_1: Conn_01x03_Pin, Connector_Phoenix_MSTB:PhoenixContact_MSTBA_2,5_3-G_1x03_P5.00mm_Horizontal, symbol Connector:Conn_01x03_Pin
- removed Motor_Logik_1: Conn_02x06_Counter_Clockwise, Connector_PinHeader_2.54mm:PinHeader_2x06_P2.54mm_Vertical_SMD, symbol Connector_Generic:Conn_02x06_Counter_Clockwise
- added Motor_Logik1: Conn_01x10_Pin, TerminalBlock_TE-Connectivity:TerminalBlock_TE_1-282834-0_1x10_P2.54mm_Horizontal, symbol Connector:Conn_01x10_Pin
- added Motor_Spannungsversorgung1: Conn_01x02_Pin, TerminalBlock_TE-Connectivity:TerminalBlock_TE_282834-2_1x02_P2.54mm_Horizontal, symbol Connector:Conn_01x02_Pin
- D2: footprint Diode_SMD:D_SMB -> Diode_SMD:D_SOD-123
Connections:
- net +24V: now also Motor_Logik1.1 (Pin_1)
- net Drehzahl_Analog_OUT: now also Motor_Logik1.10 (Pin_10)
- net GND: now also Motor_Logik1.2 (Pin_2), Motor_Spannungsversorgung1.2 (Pin_2)
- net IN0_OUT: now also D2.1 (K), Motor_Logik1.9 (Pin_9); no longer D2.1 (K)
- net IN1_OUT: now also D2.1 (K), Motor_Logik1.8 (Pin_8); no longer D2.1 (K)
- net IN2_OUT: now also D2.1 (K), Motor_Logik1.7 (Pin_7); no longer D2.1 (K)
- net IN3_OUT: now also D2.1 (K), Motor_Logik1.6 (Pin_6); no longer D2.1 (K)
- net OUT1_IN: now also D2.1 (K), Motor_Logik1.3 (Pin_3); no longer D2.1 (K)
- net OUT2_IN: now also D2.1 (K), Motor_Logik1.4 (Pin_4); no longer D2.1 (K)
- net OUT3_IN: now also D2.1 (K), Motor_Logik1.5 (Pin_5); no longer D2.1 (K)
- net at F2.1: now also Motor_Spannungsversorgung1.1 (Pin_1)
- net +5V renamed +3.3V
- no-connect marks 4 -> 1
Other:
- moved on the sheet: D2

Commit message: finished assigning pins and creating pcb
Parts:
- Motor_Spannungsversorgung1: footprint TerminalBlock_TE-Connectivity:TerminalBlock_TE_282834-2_1x02_P2.54mm_Horizontal -> TerminalBlock_Phoenix:TerminalBlock_Phoenix_PT-1,5-2-3.5-H_1x02_P3.50mm_Horizontal
Changed lines of the file:
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@@
       (effects (font (size 1.27 1.27)))
     )
-    (property "Footprint" "TerminalBlock_TE-Connectivity:TerminalBlock_TE_282834-2_1x02_P2.54mm_Horizontal" (at 24.13 30.48 0)
+    (property "Footprint" "TerminalBlock_Phoenix:TerminalBlock_Phoenix_PT-1,5-2-3.5-H_1x02_P3.50mm_Horizontal" (at 24.13 30.48 0)
       (effects (font (size 1.27 1.27)) hide)
     )
