File: pcb/Optokoppler.kicad_sch (KiCad schematic)
At the start: 27 parts, among them U10 LTV-817S, U11 LTV-817S, U3 LTV-817S, U4 LTV-817S, U5 LTV-817S, U6 LTV-817S, U7 LTV-817S, U8 LTV-817S, U9 LTV-817S

Commit message: finished assigning pins and creating pcb
Parts:
- U10, U11, U3, U4, U5, U6, U7, U8, U9: footprint Package_DIP:SMDIP-4_W9.53mm -> Package_DIP:SMDIP-4_W7.62mm
